File: Nhat.kicad_pcb (KiCad board)
At the start: 2 copper layers, 50.8 x 74.4 mm, 48 parts, among them J1 USB_C_Receptacle_USB2.0_16P, J2 Conn_01x04, J3 Conn_01x04, Q1 SS8050, Q2 SS8050, Q5 SS8550, Q6 SS8550, U1 ESP32-WROOM-32, U2 HX711, U3 HX711, U4 MPU-6050, U5 CH340C, U7 AMS1117-3.3

Commit message: update schematic, routing
Parts:
- added C17: 100nf, Capacitor_SMD:C_0603_1608Metric_Pad1.08x0.95mm_HandSolder, B.Cu at (36.6, 104.3)
- added C18: 10uf, Capacitor_SMD:C_0603_1608Metric_Pad1.08x0.95mm_HandSolder, B.Cu at (36.6, 102.8)
- added SW1: SW_Push, tue_sw_smd_3x6x2.5:tue_sw_smd_3x6x2.5mm, F.Cu at (44.0, 113.3)
- added SW2: SW_Push, tue_sw_smd_3x6x2.5:tue_sw_smd_3x6x2.5mm, F.Cu at (52.3, 113.3)
- C10, C11, C12, C13, C15, C16, C3, C5, C6, C7, C8, C9, Q1, Q2, R13, R14, R15, R16, R17, R18, R19, R21, R22, R31, R32, U5: moved to B.Cu
- C2, C4: footprint Capacitor_SMD:C_0603_1608Metric_Pad1.08x0.95mm_HandSolder -> Capacitor_Tantalum_SMD:CP_EIA-3216-12_Kemet-S_HandSolder
- moved U4 118.8 mm to (64.3, 90.8)
- moved Q2 116.3 mm to (69.3, 104.1)
- moved U7 116.3 mm to (62.8, 101.3)
- moved Q1 116.2 mm to (69.3, 100.4)
- moved R21 115.3 mm to (39.5, 92.4), turned to 90 degrees
- moved C7 113.7 mm to (47.8, 62.5), turned to 90 degrees
- moved C8 110.6 mm to (43.7, 66.6), turned to -90 degrees
- moved R15 108.6 mm to (39.4, 110.2), turned to 90 degrees
- moved C6 102.6 mm to (52.9, 71.9), turned to -90 degrees
- moved C9 102.6 mm to (53.1, 68.4), turned to -90 degrees
- moved C12 100.8 mm to (54.3, 77.6), turned to 90 degrees
- moved C13 100.4 mm to (54.3, 81.0), turned to 90 degrees
- moved C5 98.5 mm to (40.9, 110.2), turned to 90 degrees
- moved R32 97.5 mm to (62.5, 88.2)
- moved R31 97.1 mm to (62.5, 86.7)
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Connections:
- U1 pad 2: unconnected-(U1-VDD-Pad2) -> +3V3
- U1 pad 27: unconnected-(U1-IO16-Pad27) -> DOUT2_ESP
- U1 pad 28: unconnected-(U1-IO17-Pad28) -> SCK2_ESP
- U1 pad 30: unconnected-(U1-IO18-Pad30) -> SCK1_ESP
- U1 pad 31: unconnected-(U1-IO19-Pad31) -> DOUT1_ESP
- U2 pad 10: GND -> unconnected-(U2-INB+-Pad10)
- U2 pad 11: unconnected-(U2-PD_SCK-Pad11) -> SCK1_ESP
- U2 pad 12: unconnected-(U2-DOUT-Pad12) -> DOUT1_ESP
- U2 pad 9: GND -> unconnected-(U2-INB--Pad9)
- U3 pad 10: GND -> unconnected-(U3-INB+-Pad10)
- U3 pad 11: unconnected-(U3-PD_SCK-Pad11) -> SCK2_ESP
- U3 pad 12: unconnected-(U3-DOUT-Pad12) -> DOUT2_ESP
- U3 pad 9: GND -> unconnected-(U3-INB--Pad9)
Routing:
- net +3V3: track 0.00 -> 178.6 mm, vias 0 -> 12
- net ESP_BOOT0: track 0.00 -> 56.9 mm, vias 0 -> 4
- net ESP_EN: track 0.00 -> 48.7 mm, vias 0 -> 3
- net GND: track 0.00 -> 45.1 mm, vias 0 -> 17
- net Net-(J1-D--PadA7): track 0.00 -> 41.9 mm, vias 0 -> 1
- net SCL_ESP: track 0.00 -> 37.3 mm, vias 0 -> 3
- net Net-(J1-D+-PadA6): track 0.00 -> 33.1 mm, vias 0 -> 1
- net RX_CH340: track 0.00 -> 30.8 mm, vias 0 -> 6
- net RX_ESP: track 0.00 -> 29.2 mm, vias 0 -> 5
- net SDA_ESP: track 0.00 -> 28.4 mm, vias 0 -> 3
- net DOUT1_ESP: track 0.00 -> 27.7 mm
- net SCK1_ESP: track 0.00 -> 26.6 mm
- net LOAD1_E+: track 0.00 -> 16.9 mm, vias 0 -> 1
- net LOAD2_E+: track 0.00 -> 16.4 mm, vias 0 -> 1
- net +5V: track 0.00 -> 14.2 mm
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- added copper zone on B.Cu, net GND
Other:
- board size 50.8 x 74.4 mm -> 40 x 60 mm
