File: Nhat.kicad_sch (KiCad schematic)
At the start: 50 parts, among them J1 USB_C_Receptacle_USB2.0_16P, J2 Conn_01x04, J3 Conn_01x04, Q1 SS8050, Q2 SS8050, Q5 SS8550, Q6 SS8550, SW1 SW_Push, SW2 SW_Push, U1 ESP32-WROOM-32, U2 HX711, U3 HX711, U4 MPU-6050, U5 CH340C, U7 AMS1117-3.3

Commit message: update schematic, routing
Parts:
- added C17: 100nf, Capacitor_SMD:C_0603_1608Metric_Pad1.08x0.95mm_HandSolder, symbol Device:C
- added C18: 10uf, Capacitor_SMD:C_0603_1608Metric_Pad1.08x0.95mm_HandSolder, symbol Device:C
- C2, C4: footprint Capacitor_SMD:C_0603_1608Metric_Pad1.08x0.95mm_HandSolder -> Capacitor_Tantalum_SMD:CP_EIA-3216-12_Kemet-S_HandSolder
- SW1, SW2: footprint (none) -> tue_sw_smd_3x6x2.5:tue_sw_smd_3x6x2.5mm
Connections:
- net +3V3: now also U1.2 (VDD), C17.1, C18.1
- net GND: now also C17.2, C18.2; no longer U2.10 (INB+), U2.9 (INB-), U3.10 (INB+), U3.9 (INB-)
- net DOUT2_ESP: now reaches U1.27 (IO16)
- net DOUT2_ESP: now also U3.12 (DOUT)
- net SCK2_ESP: now reaches U1.28 (IO17)
- net SCK2_ESP: now also U3.11 (PD_SCK)
- net SCK1_ESP: now reaches U1.30 (IO18)
- net SCK1_ESP: now also U2.11 (PD_SCK)
- net DOUT1_ESP: now reaches U1.31 (IO19)
- net DOUT1_ESP: now also U2.12 (DOUT)
- no-connect marks 15 -> 40
Other:
- moved on the sheet: U1
