File: ws/Nhat.kicad_pcb (KiCad board)
At the start: 2 copper layers, 40 x 60 mm, 52 parts, among them J1 USB_C_Receptacle_USB2.0_16P, J2 Conn_01x04, J3 Conn_01x04, Q1 SS8050, Q2 SS8050, Q5 SS8550, Q6 SS8550, SW1 SW_Push, SW2 SW_Push, U1 ESP32-WROOM-32, U2 HX711, U3 HX711, U4 MPU-6050, U5 CH340C, U7 AMS1117-3.3

Commit message: add Led
Parts:
- added PW1: LED, Capacitor_SMD:C_0603_1608Metric_Pad1.08x0.95mm_HandSolder, F.Cu at (71.0, 97.5)
- added R20: 220, Resistor_SMD:R_0603_1608Metric_Pad0.98x0.95mm_HandSolder, F.Cu at (69.4, 97.5)
- added R33: 220, Resistor_SMD:R_0603_1608Metric_Pad0.98x0.95mm_HandSolder, F.Cu at (39.6, 87.1)
- added R34: 220, Resistor_SMD:R_0603_1608Metric_Pad0.98x0.95mm_HandSolder, F.Cu at (43.0, 87.1)
- added RX1: LED, Capacitor_SMD:C_0603_1608Metric_Pad1.08x0.95mm_HandSolder, F.Cu at (46.3, 87.1)
- added TX1: LED, Capacitor_SMD:C_0603_1608Metric_Pad1.08x0.95mm_HandSolder, F.Cu at (36.2, 87.1)
- renumbered SW2 to BOOT1, SW1 to EN1
Routing:
- net SCK1_ESP: track 26.6 -> 32.1 mm, vias 0 -> 2
- net DOUT1_ESP: track 27.7 -> 32.6 mm, vias 0 -> 2
- net GND: track 45.1 -> 49.2 mm, vias 17 -> 20
- net SCK2_ESP: track 12.2 -> 16.2 mm, vias 0 -> 2
- net DOUT2_ESP: track 10.0 -> 13.8 mm, vias 0 -> 2
- net RX_ESP: track 29.2 -> 32.2 mm
- net TX_ESP: track 1.90 -> 4.74 mm
- net +3V3: track 178.6 -> 181.4 mm
- net Net-(TX1-A): track 0.00 -> 1.59 mm
- net Net-(RX1-A): track 0.00 -> 1.59 mm
- net Net-(PW1-A): track 0.00 -> 1.58 mm
