File: ws/Nhat.kicad_sch (KiCad schematic)
At the start: 52 parts, among them J1 USB_C_Receptacle_USB2.0_16P, J2 Conn_01x04, J3 Conn_01x04, Q1 SS8050, Q2 SS8050, Q5 SS8550, Q6 SS8550, SW1 SW_Push, SW2 SW_Push, U1 ESP32-WROOM-32, U2 HX711, U3 HX711, U4 MPU-6050, U5 CH340C, U7 AMS1117-3.3

Commit message: add Led
Parts:
- added PW1, RX1, TX1: LED, Capacitor_SMD:C_0603_1608Metric_Pad1.08x0.95mm_HandSolder, symbol Device:LED
- added R20, R33, R34: 220, Resistor_SMD:R_0603_1608Metric_Pad0.98x0.95mm_HandSolder, symbol Device:R
- renumbered SW2 to BOOT1, SW1 to EN1
Connections:
- net +3V3: now also R20.1
- net GND: now also PW1.1 (K), RX1.1 (K), TX1.1 (K)
- net RX_ESP: now also R34.1
- net TX_ESP: now also R33.1
- new net: PW1.2 (A), R20.2
- new net: R34.2, RX1.2 (A)
- new net: R33.2, TX1.2 (A)
Other:
- moved on the sheet: C17, C18
